File: VL160.kicad_pcb (KiCad board)
At the start: 4 copper layers, 24 x 14 mm, 12 parts, among them J1 USB_C_Receptacle, J2 USB3_A, U1 VL160, U2 LM3480-5.0

Commit message: Sync 2022/01/07 周五 16:48:22.07
Parts:
- moved R3 2.24 mm to (142.9, 94.5), turned to 0 degrees
- moved R5 1.88 mm to (142.9, 91.8), turned to 0 degrees
- moved R4 0.74 mm to (142.9, 93.1), turned to 0 degrees
Routing:
- net Net-(R5-Pad2): track 0.00 -> 6.81 mm
- net /D+: track 16.4 -> 21.2 mm
- net Net-(R4-Pad2): track 0.00 -> 4.61 mm
- net VBUS: track 4.30 -> 8.71 mm
- net /D-: track 19.1 -> 22.1 mm
- net Net-(R3-Pad2): track 0.00 -> 2.79 mm
- net GND: vias 0 -> 1
- net (no net): vias 0 -> 2

Commit message: Sync 2022/01/11 周二 21:14:02.89
Parts:
- added H1: MountingHole, VL160:Hole_1.152mm_JLCSMT, F.Cu at (137.4, 102.6)
- added H2: MountingHole, VL160:Hole_1.152mm_JLCSMT, F.Cu at (155.3, 99.8)
- added H3: MountingHole, VL160:Hole_1.152mm_JLCSMT, F.Cu at (145.3, 91.1)
- J1, J2: moved to B.Cu
- U2: value LM3480-5.0 -> SE8550
- moved C2 5.65 mm to (140.1, 93.1), turned to 180 degrees
- moved C3 4.97 mm to (140.1, 94.5), turned to 180 degrees
- moved C1 4.83 mm to (134.5, 91.6), turned to 90 degrees
- moved J1 3.39 mm to (135.2, 93.6)
- moved U2 1.86 mm to (136.9, 92.0), turned to 180 degrees
- moved J2 1.47 mm to (148.7, 98.3), turned to 0 degrees
Connections:
- U1 pad 29: (no net) -> GND
- U2 pad 1: VCC -> GND
- U2 pad 2: VBUS -> VCC
- U2 pad 3: GND -> VBUS
Routing:
- net VBUS: track 8.71 -> 39.0 mm, vias 2 -> 5
- net VCC: track 0.00 -> 12.7 mm
- net /CC2: track 6.99 -> 8.77 mm
- net /CC1: track 6.11 -> 6.83 mm
- net GND: vias 1 -> 24
- net (no net): vias 2 -> 0
- added copper zone on B.Cu, net GND
- added copper zone on F.Cu, net GND
- added copper zone on In1.Cu, net GND
- added copper zone on In2.Cu, net GND
Other:
- net class 90R_IN: via_dia 0.4 -> 0.45
- net class 90R_OUT: via_dia 0.4 -> 0.45
- net class Default: via_dia 0.4 -> 0.45
- net class POWER: via_dia 0.5 -> 0.45; via_drill 0.3 -> 0.2
- rule via_min_drill: 0 -> 0.2
- rule via_min_size: 0 -> 0.45

Commit message: Sync 2022/01/19 周三 11:41:49.34
Parts:
- added TP1: TestPoint, VL160:TestPoint_Pad_D0.7mm, F.Cu at (141.1, 102.1)
- added TP2: TestPoint, VL160:TestPoint_Pad_D0.7mm, F.Cu at (142.5, 102.1)
- added TP3: TestPoint, VL160:TestPoint_Pad_D0.7mm, F.Cu at (143.9, 102.1)
- added TP4: TestPoint, VL160:TestPoint_Pad_D0.7mm, F.Cu at (145.2, 101.0)
- added TP5: TestPoint, VL160:TestPoint_Pad_D0.7mm, F.Cu at (145.2, 102.5)
- J1: footprint VL160:USB-C-SMD_TYPE-C-31-G-01 -> Connector_USB:USB_C_Receptacle_Amphenol_12401548E4-2A; moved to F.Cu
- moved H1 6.87 mm to (130.6, 103.0)
- moved J1 5.68 mm to (130.8, 97.2), turned to 270 degrees
- moved R2 2.89 mm to (139.7, 102.4), turned to 270 degrees
- moved R1 1.48 mm to (138.3, 102.4)
- moved U2 0.48 mm to (137.3, 91.7)
- moved C1 0.43 mm to (134.4, 91.2), turned to 180 degrees
Connections:
- U1 pad 11: (no net) -> Net-(TP1-Pad1)
- U1 pad 12: (no net) -> Net-(TP2-Pad1)
- U1 pad 14: (no net) -> Net-(TP3-Pad1)
- U1 pad 15: (no net) -> Net-(TP5-Pad1)
- U1 pad 16: (no net) -> Net-(TP4-Pad1)
Routing:
- net /CC2: track 8.77 -> 17.8 mm
- net VBUS: track 39.0 -> 30.4 mm, vias 5 -> 4
- net Net-(R2-Pad1): track 1.32 -> 6.97 mm
- net Net-(TP5-Pad1): track 0.00 -> 3.00 mm
- net /CC1: track 6.83 -> 4.48 mm, vias 1 -> 2
- net Net-(TP4-Pad1): track 0.00 -> 2.32 mm
- net Net-(TP3-Pad1): track 0.00 -> 2.31 mm
- net Net-(TP2-Pad1): track 0.00 -> 1.99 mm
- net /TX1+: track 6.67 -> 5.02 mm, vias 1 -> 0
- net /TX1-: track 6.67 -> 5.02 mm, vias 1 -> 0
- net Net-(R1-Pad1): track 1.12 -> 2.63 mm
- net Net-(TP1-Pad1): track 0.00 -> 1.49 mm
- net /RX2+: track 5.62 -> 4.35 mm, vias 1 -> 0
- net /RX2-: track 5.62 -> 4.35 mm, vias 1 -> 0
- net /RX1+: track 8.42 -> 9.43 mm, vias 0 -> 1
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Other:
- board size 24 x 14 mm -> 30 x 14 mm
